Commit message: solid2urdf

File: solidworks/blattoidea/urdf/blattoidea.urdf (robot description, URDF)
Before this commit: robot blattoidea, 7 links, 6 joints
Joints:
- joint lw_joint: origin xyz=-0.0066026 -0.41814 0.15635 rpy=-2.8253 0 -1.5708 -> xyz=-0.022603 -0.41814 0.15635 rpy=2.2379 0 -1.5708
