Commit message: urdf

File: blattoidea/urdf/blattoidea.urdf (robot description, URDF)
Before this commit: robot blattoidea, 7 links, 6 joints
Links:
- added link lc_segment_Link, mass 0; collision mesh filename=package://blattoidea/meshes/lc_segment_Link.STL; visual mesh filename=package://blattoidea/meshes/lc_segment_Link.STL
- added link rc_segment_Link, mass 0.045681; collision mesh filename=package://blattoidea/meshes/rc_segment_Link.STL; visual mesh filename=package://blattoidea/meshes/rc_segment_Link.STL
- link base_link: mass 3.6045 -> 8.7926
- link l_caster_Link: mass 0.026461 -> 0.0264605807216404
- link r_caster_Link: mass 0.026461 -> 0.0264605676973988
- link rc_wheel_Link: mass 0.0499 -> 0.0498995656286702
Joints:
- added joint lc_segment_joint: type fixed, parent base_link, child lc_segment_Link, origin xyz=0.18405 0.053 -0.13557 rpy=-0.052561 -1.4732 3.1416, axis 0 0 0
- added joint rc_segment_joint: type fixed, parent base_link, child rc_segment_Link, origin xyz=0.13468 0.053 0.13557 rpy=3.089 1.4732 0, axis 0 0 0
- joint l_caster_joint: origin xyz=0.3079 -0.43554 0.089119 rpy=1.5182 0 1.0025 -> xyz=-0.002 0.0013134 -0.024965 rpy=0.014242 -0.66482 -0.041251; parent base_link -> lc_segment_Link
- joint lc_wheel_joint: axis 1 0 0 -> -1 0 0; origin xyz=-0.002 0.010904 0.025608 rpy=-1.5211 0 -3.1416 -> xyz=0 -0.0013134 0.024965 rpy=-2.8657 0 -3.1416
- joint lw_joint: origin xyz=-0.022603 -0.41814 0.15635 rpy=2.2379 0 -1.5708 -> xyz=-0.17114 -0.002 -0.089756 rpy=-2.9986 1.5708 -1.6213
- joint r_caster_joint: origin xyz=0.3079 -0.15554 0.089119 rpy=1.5182 0 1.7592 -> xyz=-0.002 0.0013134 -0.024965 rpy=3.0363 -0.090647 -3.1368; parent base_link -> rc_segment_Link
- joint rc_wheel_joint: origin xyz=-0.002 0.010904 0.025608 rpy=2.3039 0 3.1416 -> xyz=0 -0.0013134 0.024965 rpy=0.1671 0 -3.1416
- joint rw_joint: origin xyz=-0.022603 -0.061936 0.15635 rpy=2.5982 0 1.5708 -> xyz=-0.17114 -0.002 0.091417 rpy=3.076 -1.5708 0

Commit message: update

File: blattoidea/urdf/blattoidea.urdf (robot description, URDF)
Before this commit: robot blattoidea, 9 links, 8 joints
Links:
- link base_link: mass 8.7926 -> 8.79255713417749
- link l_caster_Link: mass 0.0264605807216404 -> 0.0264605949467887
- link lc_segment_Link: mass 0 -> 0.0456806083099005
- link lc_wheel_Link: mass 0.0499 -> 0.0498995656286702
- link lw_Link: mass 0.97717 -> 0.977168759094327
- link r_caster_Link: mass 0.0264605676973988 -> 0.0264605949467884
- link rc_segment_Link: mass 0.045681 -> 0.0456806083099006
- link rc_wheel_Link: mass 0.0498995656286702 -> 0.0498995656286701
- link rw_Link: mass 0.97717 -> 0.977168759094327
Joints:
- joint l_caster_joint: axis 0 1 0 -> 0 0.99862 0.052537; origin xyz=-0.002 0.0013134 -0.024965 rpy=0.014242 -0.66482 -0.041251 -> xyz=-0.002 0.0013134 -0.024965 rpy=0.00025094 -0.097478 -0.0051446
- joint lc_segment_joint: origin xyz=0.18405 0.053 -0.13557 rpy=-0.052561 -1.4732 3.1416 -> xyz=-0.18405 0.13557 -0.053 rpy=1.5182 0 -1.4732
- joint lc_wheel_joint: origin xyz=0 -0.0013134 0.024965 rpy=-2.8657 0 -3.1416 -> xyz=0 -0.0013134 0.024965 rpy=3.089 0 3.1416
- joint lw_joint: origin xyz=-0.17114 -0.002 -0.089756 rpy=-2.9986 1.5708 -1.6213 -> xyz=0.17114 0.1226 0.002 rpy=-1.5708 0 1.5708
- joint r_caster_joint: axis 0 1 0 -> 0 0.99862 0.052537; origin xyz=-0.002 0.0013134 -0.024965 rpy=3.0363 -0.090647 -3.1368 -> xyz=-0.002 0.0013134 -0.024965 rpy=3.0362 0.097478 3.1364
- joint rc_segment_joint: origin xyz=0.13468 0.053 0.13557 rpy=3.089 1.4732 0 -> xyz=-0.13468 -0.13557 -0.053 rpy=1.5182 0 1.6684
- joint rc_wheel_joint: origin xyz=0 -0.0013134 0.024965 rpy=0.1671 0 -3.1416 -> xyz=0 -0.0013134 0.024965 rpy=-0.052561 0 3.1416
- joint rw_joint: origin xyz=-0.17114 -0.002 0.091417 rpy=3.076 -1.5708 0 -> xyz=0.17114 -0.1226 0.002 rpy=1.5708 0 -1.5708

Commit message: update

File: blattoidea/urdf/blattoidea.urdf (robot description, URDF)
Before this commit: robot blattoidea, 9 links, 8 joints
Links:
- link l_caster_Link: mass 0.0264605949467887 -> 0.0264605949467886
- link rw_Link: mass 0.977168759094327 -> 0.977168759094326
Joints:
- joint l_caster_joint: axis 0 0.99862 0.052537 -> 0 0.99861896542272 0.052537242962078; origin xyz=-0.002 0.0013134 -0.024965 rpy=0.00025094 -0.097478 -0.0051446 -> xyz=-0.00199999999996087 0.00131343107405134 -0.0249654741355564 rpy=0.00025094260002981 -0.0974777924807896 -0.00514462437867282
- joint lc_segment_joint: origin xyz=-0.18405 0.13557 -0.053 rpy=1.5182 0 -1.4732 -> xyz=-0.184049370454713 0.135573068545923 -0.0529999999999954 rpy=1.51823488521493 0 -1.47318329844307
- joint lc_wheel_joint: origin xyz=0 -0.0013134 0.024965 rpy=3.089 0 3.1416 -> xyz=0 -0.00131343107400735 0.0249654741355546 rpy=3.08903121200983 0 3.14159265358979
- joint lw_joint: origin xyz=0.17114 0.1226 0.002 rpy=-1.5708 0 1.5708 -> xyz=0.171136704119859 0.122599999999968 0.00200000000000291 rpy=-1.5707963267949 0 1.5707963267949
- joint r_caster_joint: axis 0 0.99862 0.052537 -> 0 0.99861896542272 0.052537242962078; origin xyz=-0.002 0.0013134 -0.024965 rpy=3.0362 0.097478 3.1364 -> xyz=-0.00200000000001023 0.00131343107405157 -0.0249654741355608 rpy=3.03621882782983 0.0974777924807896 3.13644802921112
- joint rc_segment_joint: origin xyz=-0.13468 -0.13557 -0.053 rpy=1.5182 0 1.6684 -> xyz=-0.134677221305586 -0.13557306854595 -0.0529999999999956 rpy=1.51823488521493 0 1.66840935514672
- joint rc_wheel_joint: origin xyz=0 -0.0013134 0.024965 rpy=-0.052561 0 3.1416 -> xyz=0 -0.0013134310740316 0.0249654741355853 rpy=-0.0525614415799654 0 3.14159265358979
- joint rw_joint: origin xyz=0.17114 -0.1226 0.002 rpy=1.5708 0 -1.5708 -> xyz=0.171136704119851 -0.122600000000032 0.00199999999999654 rpy=1.5707963267949 0 -1.5707963267949

Commit message: update

File: blattoidea/urdf/blattoidea.urdf (robot description, URDF)
Before this commit: robot blattoidea, 9 links, 8 joints
Links:
- added link base_footprint
- added link camera_depth_frame, mass 0.01
- added link camera_depth_optical_frame, mass 0.001
- added link camera_link, mass 0.01; collision box size=0.0730 .2760 0.0720; visual mesh filename=package://blattoidea/meshes/kinect.dae
- added link camera_rgb_frame, mass 0.001
- added link camera_rgb_optical_frame, mass 0.001
Joints:
- added joint base_camera_joint: type fixed, parent base_link, child camera_link, origin xyz=0.2 0 0.17 rpy=0 0 0
- added joint base_footprint_base_link_joint: type fixed, parent base_footprint, child base_link, origin xyz=0 0 -15
- added joint camera_depth_joint: type fixed, parent camera_link, child camera_depth_frame, origin xyz=0 0.011 0 rpy=0 0 0
- added joint camera_depth_optical_joint: type fixed, parent camera_depth_frame, child camera_depth_optical_frame, origin xyz=0 0 0 rpy=-1.57 0 -1.57
- added joint camera_rgb_joint: type fixed, parent camera_link, child camera_rgb_frame, origin xyz=0 -0.012 0 rpy=0 0 0
- added joint camera_rgb_optical_joint: type fixed, parent camera_rgb_frame, child camera_rgb_optical_frame, origin xyz=0 0 0 rpy=-1.57 0 -1.57
- joint rw_joint: axis 1 0 0 -> -1 0 0

Commit message: gazebo service set model vel

File: blattoidea/urdf/blattoidea.urdf (robot description, URDF)
Before this commit: robot blattoidea, 15 links, 14 joints
Joints:
- joint base_footprint_base_link_joint: origin xyz=0 0 -15 -> xyz=0 0 0.20

Commit message: update

File: blattoidea/urdf/blattoidea.urdf (robot description, URDF)
Before this commit: robot blattoidea, 15 links, 14 joints
Links:
- removed link lc_segment_Link
- removed link rc_segment_Link
- link base_link: mass 8.79255713417749 -> 3.1167
- link l_caster_Link: mass 0.0264605949467886 -> 0.026461
- link lc_wheel_Link: mass 0.0498995656286702 -> 0.0499
- link lw_Link: mass 0.977168759094327 -> 0.97717
- link r_caster_Link: mass 0.0264605949467884 -> 0.026461
- link rc_wheel_Link: mass 0.0498995656286701 -> 0.0499
- link rw_Link: mass 0.977168759094326 -> 0.97717
Joints:
- removed joint lc_segment_joint
- removed joint rc_segment_joint
- joint l_caster_joint: axis 0 0.99861896542272 0.052537242962078 -> 0 0.99862 0.052537; origin xyz=-0.00199999999996087 0.00131343107405134 -0.0249654741355564 rpy=0.00025094260002981 -0.0974777924807896 -0.00514462437867282 -> xyz=-0.15936 0.14 -0.0051144 rpy=1.5182 0 -1.5708; parent lc_segment_Link -> base_link
- joint lc_wheel_joint: origin xyz=0 -0.00131343107400735 0.0249654741355546 rpy=3.08903121200983 0 3.14159265358979 -> xyz=0 -0.049133 0.02245 rpy=3.089 0 3.1416
- joint lw_joint: origin xyz=0.171136704119859 0.122599999999968 0.00200000000000291 rpy=-1.5707963267949 0 1.5707963267949 -> xyz=0.17114 0.1226 -0.006 rpy=-1.5708 0 1.5708
- joint r_caster_joint: axis 0 0.99861896542272 0.052537242962078 -> 0 0.99862 0.052537; origin xyz=-0.00200000000001023 0.00131343107405157 -0.0249654741355608 rpy=3.03621882782983 0.0974777924807896 3.13644802921112 -> xyz=-0.15936 -0.14 -0.0051144 rpy=1.5182 0 -1.5708; parent rc_segment_Link -> base_link
- joint rc_wheel_joint: origin xyz=0 -0.0013134310740316 0.0249654741355853 rpy=-0.0525614415799654 0 3.14159265358979 -> xyz=0 -0.049133 0.02245 rpy=-0.052561 0 3.1416
- joint rw_joint: axis -1 0 0 -> 1 0 0; origin xyz=0.171136704119851 -0.122600000000032 0.00199999999999654 rpy=1.5707963267949 0 -1.5707963267949 -> xyz=0.17114 -0.1226 -0.006 rpy=1.5708 0 -1.5708

Commit message: update dlattoidea

File: blattoidea/urdf/blattoidea.urdf (robot description, URDF)
Before this commit: robot blattoidea, 13 links, 12 joints
Joints:
- joint rw_joint: axis 1 0 0 -> -1 0 0

Commit message: update catch ball

File: blattoidea/urdf/blattoidea.urdf (robot description, URDF)
Before this commit: robot blattoidea, 15 links, 14 joints
Joints:
- joint base_camera_joint: origin xyz=0.2 0 0.17 rpy=0 0 0 -> xyz=0.0 0.17 0.17 rpy=0 0 1.57
- joint camera_depth_joint: origin xyz=0 0.011 0 rpy=0 0 0 -> xyz=0 0.011 0 rpy=0 0 1.57

Commit message: up

File: blattoidea/urdf/blattoidea.urdf (robot description, URDF)
Before this commit: robot blattoidea, 15 links, 14 joints
Joints:
- joint base_camera_joint: origin xyz=0.0 0.17 0.17 rpy=0 0 1.57 -> xyz=0.2 0.0 0.17 rpy=0 0 0
- joint camera_depth_joint: origin xyz=0 0.011 0 rpy=0 0 1.57 -> xyz=0 0.011 0 rpy=0 0 0
- joint camera_depth_optical_joint: origin xyz=0 0 0 rpy=-1.57 0 -1.57 -> xyz=0 0 0 rpy=-1.57 0 0
- joint camera_rgb_optical_joint: origin xyz=0 0 0 rpy=-1.57 0 -1.57 -> xyz=0 0 0 rpy=-1.57 0 0

File: blattoidea/urdf/kinect.xacro (robot description, xacro)
@@ -3,5 +3,5 @@
 	<xacro:macro name="kinect">
 			<joint name="base_camera_joint" type="fixed">
-				<origin xyz="0.0 0.17 0.17" rpy="0 0 1.57" />
+				<origin xyz="0.17 0.0 0.17" rpy="0 0 0" />
 				<parent link="base_link" />
 				<origin xyz="0 0 0" rpy="0 0 0" />
