Commit message: update

File: blattoidea/urdf/GPS.xacro (robot description, xacro)
@@ -10,5 +10,5 @@
 		<link name="GPS_link">
 		</link>
-		<gazebo reference="GPS_link">
+		<gazebo>
 				<plugin name="gps_controller" filename="libhector_gazebo_ros_gps.so">
 					<alwayson>true</alwayson>

File: blattoidea/urdf/base_footprint.xacro (robot description, xacro)
@@ -5,5 +5,5 @@
 		</link>
 		<joint name="base_footprint_base_link_joint" type="fixed">
-			<origin xyz="0 0 0.20"/>
+			<origin xyz="0 0 0.08255"/>
 			<parent link="base_footprint"/>
 			<child link="base_link"/>

File: blattoidea/urdf/blattoidea.urdf.xacro (robot description, xacro)
@@ -374,17 +374,6 @@
       <dynamics damping="0.0" friction="0.0"/>
   </joint>
+	<gazebo>
      <plugin name="JointStatePublisher" filename="libJointStatePublisher.so"/>
-  <gazebo>
-     <plugin name="gps_controller" filename="libhector_gazebo_ros_gps.so">
-      <alwayson>true</alwayson>
-      <updaterate>1.0</updaterate>
-      <bodyname>base_link</bodyname>
-      <topicname>/fix</topicname>
-      <velocitytopicname>/fix_velocity</velocitytopicname>
-      <drift>5.0 5.0 5.0</drift>
-      <gaussiannoise>0.1 0.1 0.1</gaussiannoise>
-      <velocitydrift>0 0 0</velocitydrift>
-      <velocitygaussiannoise>0.1 0.1 0.1</velocitygaussiannoise>
-    </plugin>
-  </gazebo>
+	</gazebo>
 </robot>

File: blattoidea/urdf/blattoidea_gazebo.urdf.xacro (robot description, xacro)
@@ -12,4 +12,6 @@
 	<xacro:include filename="$(find blattoidea)/urdf/kinect.xacro"/>
 	<xacro:kinect/>
+	<xacro:include filename="$(find blattoidea)/urdf/GPS.xacro"/>
+	<xacro:GPS/>
 	<!-- <xacro:include filename="$(find blattoidea)/urdf/camera.xacro"/>
 	<xacro:rgb_camera/> -->
