Commit message: update

File: blattoidea/urdf/base_footprint.xacro (robot description, xacro)
@@ -6,6 +6,6 @@
 		<joint name="base_footprint_base_link_joint" type="fixed">
 			<origin xyz="0 0 0.20"/>
-			<parent link="base_link"/>
-			<child link="base_footprint"/>
+			<parent link="base_footprint"/>
+			<child link="base_link"/>
 		</joint>
 	</xacro:macro>

File: blattoidea/urdf/kinect.xacro (robot description, xacro)
@@ -3,9 +3,9 @@
 	<xacro:macro name="kinect">
 		<joint name="base_camera_joint" type="fixed">
-				<axis xyz="1 0 0" />
-				<origin xyz="0.17 0.0 0.17" rpy="0 0 0" />
-				<parent link="base_link" />
-				<child link="camera_link" />
-			  </joint>
+			<origin xyz="0.2 0 0.17" rpy="0 0 0" />
+			<parent link="base_link" />
+			<origin xyz="0 0 0" rpy="0 0 0" />
+			<child link="camera_link" />
+		</joint>
 		<link name="camera_link">
 			<inertial>
@@ -29,10 +29,60 @@
 			</collision>
 		</link>
-		<joint name="camera_optical_joint" type="fixed">
-			<origin xyz="0 0 0" rpy="-1 -1 -1" />
+		<joint name="camera_depth_joint" type="fixed">
+			<origin xyz="0 0.011 0" rpy="0 0 0" />
+				<parent link="camera_link" />
+			<child link="camera_depth_frame" />
+		</joint>
+		<link name="camera_depth_frame">
+			<inertial>
+				<mass value="0.01" />
+				<origin xyz="0 0 0" />
+				<inertia ixx="0.001" ixy="0.0" ixz="0.0"
+					iyy="0.001" iyz="0.0"
+					izz="0.001" />
+			</inertial>
+		</link>
+		<joint name="camera_depth_optical_joint" type="fixed">
+			<origin xyz="0 0 0" rpy="-1.57 0 -1.57" />
+			<parent link="camera_depth_frame" />
+			<child link="camera_depth_optical_frame" />
+		</joint>
+		<link name="camera_depth_optical_frame">
+			<inertial>
+				<mass value="0.001" />
+				<origin xyz="0 0 0" />
+				<inertia ixx="0.0001" ixy="0.0" ixz="0.0"
+					iyy="0.0001" iyz="0.0"
+					izz="0.0001" />
+			</inertial>
+		</link>
+		<joint name="camera_rgb_joint" type="fixed">
+			<origin xyz="0 -0.012 0" rpy="0 0 0" />
 			<parent link="camera_link" />
-			<child link="camera_optical_frame" />
+			<child link="camera_rgb_frame" />
 		</joint>
-		<link name="camera_optical_frame"/>
+		<link name="camera_rgb_frame">
+			<inertial>
+				<mass value="0.001" />
+				<origin xyz="0 0 0" />
+				<inertia ixx="0.0001" ixy="0.0" ixz="0.0"
+					iyy="0.0001" iyz="0.0"
+					izz="0.0001" />
+			</inertial>
+		</link>
+		<joint name="camera_rgb_optical_joint" type="fixed">
+			<origin xyz="0 0 0" rpy="-1.57 0 -1.57" />
+			<parent link="camera_rgb_frame" />
+			<child link="camera_rgb_optical_frame" />
+		</joint>
+		<link name="camera_rgb_optical_frame">
+			<inertial>
+			<mass value="0.001" />
+			<origin xyz="0 0 0" />
+			<inertia ixx="0.0001" ixy="0.0" ixz="0.0"
+				iyy="0.0001" iyz="0.0"
+				izz="0.0001" />
+			</inertial>
+		</link>
 		<gazebo reference="camera_link">
 			<sensor name="kinect" type="depth">
@@ -60,5 +110,5 @@
 					<depthImageInfoTopicName>/kinect/depth/camera_info</depthImageInfoTopicName>
 					<pointCloudTopicName>/kinect/depth/points</pointCloudTopicName>
-					<frameName>camera_optical_frame</frameName>
+					<frameName>camera_link</frameName>
 					<pointCloudCutoff>0.05</pointCloudCutoff>
 					<pointCloudCutoffMax>20</pointCloudCutoffMax>

Commit message: u

File: blattoidea/urdf/base_footprint.xacro (robot description, xacro)
@@ -5,5 +5,5 @@
 		</link>
 		<joint name="base_footprint_base_link_joint" type="fixed">
-			<origin xyz="0 0 0.08255"/>
+			<origin xyz="0 0 0.08256"/>
 			<parent link="base_footprint"/>
 			<child link="base_link"/>
