Commit message: update

File: blattoidea/urdf/DiffDrive.xacro (robot description, xacro)
@@ -29,6 +29,6 @@
 				<leftJoint>lw_joint</leftJoint>
 				<rightJoint>rw_joint</rightJoint>
-				<wheelSeparation>0.34</wheelSeparation>
-				<wheelDiameter>0.165</wheelDiameter>
+				<wheelSeparation>0.44</wheelSeparation>
+				<wheelDiameter>0.1651</wheelDiameter>
 				<torque>1.41</torque>
 				<commandTopic>cmd_vel</commandTopic>

File: blattoidea/urdf/base_footprint.xacro (robot description, xacro)
@@ -6,6 +6,6 @@
 		<joint name="base_footprint_base_link_joint" type="fixed">
 			<origin xyz="0 0 0.20"/>
-			<parent link="base_footprint"/>
-			<child link="base_link"/>
+			<parent link="base_link"/>
+			<child link="base_footprint"/>
 		</joint>
 	</xacro:macro>

File: blattoidea/urdf/blattoidea.urdf.xacro (robot description, xacro)
@@ -5,6 +5,11 @@
 <robot xmlns:xacro="http://www.ros.org/wiki/xacro"
 	name="blattoidea">
-  <link
-    name="base_link">
+<link name="base_link" />
+<joint name="base_link_to_chassis" type="fixed">
+    <parent link="base_link"/>
+    <child link="chassis"/>
+  </joint>
+  <link
+    name="chassis">
     <inertial>
       <origin
@@ -363,3 +368,78 @@
       xyz="-1 0 0" />
   </joint>
+<joint name="base_camera_joint" type="fixed">
+				<axis xyz="1 0 0" />
+				<origin xyz="0.17 0.0 0.17" rpy="0 0 0" />
+				<parent link="base_link" />
+				<child link="camera_link" />
+			  </joint>
+		<link name="camera_link">
+			<inertial>
+				<mass value="0.01" />
+				<origin xyz="0 0 0" />
+				<inertia ixx="0.001" ixy="0.0" ixz="0.0"
+					iyy="0.001" iyz="0.0"
+					izz="0.001" />
+			</inertial>
+				<visual>
+				<origin xyz=" 0 0 0 " rpy="0 0 0" />
+				<geometry>
+					<mesh filename="package://blattoidea/meshes/kinect.dae"/>
+				</geometry>
+			</visual>
+			<collision>
+				<origin xyz="0.0 0.0 0.0" rpy="0 0 0" />
+				<geometry>
+					<box size="0.0730 .2760 0.0720"/>
+				</geometry>
+			</collision>
+		</link>
+		<joint name="camera_optical_joint" type="fixed">
+			<origin xyz="0 0 0" rpy="-1.57 0 -1.57" />
+			<parent link="camera_link" />
+			<child link="camera_optical_frame" />
+		</joint>
+		<link name="camera_optical_frame"/>
+		<gazebo reference="camera_optical_frame"/>
+		<gazebo reference="camera_link">
+			<sensor name="kinect" type="depth">
+				<update_rate>30</update_rate>
+				<camera>
+					<horizontal_fov>1.047198</horizontal_fov>
+					<image>
+						<width>640</width>
+						<height>480</height>
+						<format>R8G8B8</format>
+					</image>
+					<clip>
+						<near>0.05</near>
+						<far>20</far>
+					</clip>
+				</camera>
+				<plugin name="depth_controller" filename="libgazebo_ros_openni_kinect.so">
+					<baseline>0.2</baseline>
+					<alwaysOn>true</alwaysOn>
+					<updateRate>30.0</updateRate>
+					<cameraName>kinect_ir</cameraName>
+					<imageTopicName>/kinect/color/image_raw</imageTopicName>
+					<cameraInfoTopicName>/kinect/color/camera_info</cameraInfoTopicName>
+					<depthImageTopicName>/kinect/depth/image_raw</depthImageTopicName>
+					<depthImageInfoTopicName>/kinect/depth/camera_info</depthImageInfoTopicName>
+					<pointCloudTopicName>/kinect/depth/points</pointCloudTopicName>
+					<frameName>camera_optical_frame</frameName>
+					<pointCloudCutoff>0.05</pointCloudCutoff>
+					<pointCloudCutoffMax>20</pointCloudCutoffMax>
+					<distortionK1>0.0</distortionK1>
+					<distortionK2>0.0</distortionK2>
+					<distortionK3>0.0</distortionK3>
+					<distortionT1>0.0</distortionT1>
+					<distortionT2>0.0</distortionT2>
+					<CxPrime>0</CxPrime>
+					<Cx>0</Cx>
+					<Cy>0</Cy>
+					<focalLength>0</focalLength>
+					<hackBaseline>0</hackBaseline>
+				</plugin>
+			</sensor>
+		</gazebo>
 </robot>

File: blattoidea/urdf/blattoidea_gazebo.urdf.xacro (robot description, xacro)
@@ -10,6 +10,8 @@
 	<xacro:include filename="$(find blattoidea)/urdf/DiffDrive.xacro"/>
 	<xacro:DiffDrive/>
-	<xacro:include filename="$(find blattoidea)/urdf/kinect.xacro"/>
-	<xacro:kinect/>
+	<!--<xacro:include filename="$(find blattoidea)/urdf/kinect.xacro"/>
+	<xacro:kinect/>-->
+	<!--<xacro:include filename="$(find blattoidea)/urdf/camera.xacro"/>
+	<xacro:rgb_camera/>-->
 	<xacro:include filename="$(find blattoidea)/urdf/hokuyo.xacro"/>
 	<xacro:laser name="base_laser" parent="base_link" xyz="0.17 0.0 0.085" rpy="3.14 0 0" meshes="package://gazebo_plugins/test/multi_robot_scenario/meshes/laser"/>

File: blattoidea/urdf/hokuyo.xacro (robot description, xacro)
@@ -36,13 +36,13 @@
                 <!-- The URG-04LX-UG01  has  683 steps with 0.35139 Degree resolution -->
                 <resolution>1</resolution>
-                <max_angle>2.0944</max_angle> <!-- 120 Degree -->
-                <min_angle>-2.0944</min_angle> <!-- -120 Degree -->
-                <samples>683</samples>
+                <max_angle>2</max_angle> <!-- 120 Degree -->
+                <min_angle>-2</min_angle> <!-- -120 Degree -->
+                <samples>720</samples>
               </horizontal>
             </scan>
             <range>
-              <min>0.08</min>
-              <max>5</max>
-              <resolution>0.01</resolution>
+              <min>0.2</min>
+              <max>10</max>
+              <resolution>0.02</resolution>
             </range>
           </ray>
@@ -56,5 +56,5 @@
           -->
           <always_on>1</always_on>
-          <update_rate>30</update_rate>
+          <update_rate>15</update_rate>
           <visualize>true</visualize>
         </sensor>

File: blattoidea/urdf/kinect.xacro (robot description, xacro)
@@ -2,8 +2,8 @@
 <robot xmlns:xacro="http://www.ros.org/wiki/xacro">
 	<xacro:macro name="kinect">
-			<joint name="base_camera_joint" type="fixed">
+		<joint name="base_camera_joint" type="fixed">
+				<axis xyz="1 0 0" />
 				<origin xyz="0.17 0.0 0.17" rpy="0 0 0" />
 				<parent link="base_link" />
-				<origin xyz="0 0 0" rpy="0 0 0" />
 				<child link="camera_link" />
 			  </joint>
@@ -29,60 +29,10 @@
 			</collision>
 		</link>
-		<joint name="camera_depth_joint" type="fixed">
-			<origin xyz="0 0.011 0" rpy="0 0 0" />
-				<parent link="camera_link" />
-			<child link="camera_depth_frame" />
+		<joint name="camera_optical_joint" type="fixed">
+			<origin xyz="0 0 0" rpy="-1 -1 -1" />
+			<parent link="camera_link" />
+			<child link="camera_optical_frame" />
 		</joint>
-		<link name="camera_depth_frame">
-			<inertial>
-				<mass value="0.01" />
-				<origin xyz="0 0 0" />
-				<inertia ixx="0.001" ixy="0.0" ixz="0.0"
-					iyy="0.001" iyz="0.0"
-					izz="0.001" />
-			</inertial>
-		</link>
-		<joint name="camera_depth_optical_joint" type="fixed">
-			<origin xyz="0 0 0" rpy="-1.57 0 -1.57" />
-			<parent link="camera_depth_frame" />
-			<child link="camera_depth_optical_frame" />
-		</joint>
-		<link name="camera_depth_optical_frame">
-			<inertial>
-				<mass value="0.001" />
-				<origin xyz="0 0 0" />
-				<inertia ixx="0.0001" ixy="0.0" ixz="0.0"
-					iyy="0.0001" iyz="0.0"
-					izz="0.0001" />
-			</inertial>
-		</link>
-		<joint name="camera_rgb_joint" type="fixed">
-			<origin xyz="0 -0.012 0" rpy="0 0 0" />
-			<parent link="camera_link" />
-			<child link="camera_rgb_frame" />
-		</joint>
-		<link name="camera_rgb_frame">
-			<inertial>
-				<mass value="0.001" />
-				<origin xyz="0 0 0" />
-				<inertia ixx="0.0001" ixy="0.0" ixz="0.0"
-					iyy="0.0001" iyz="0.0"
-					izz="0.0001" />
-			</inertial>
-		</link>
-		<joint name="camera_rgb_optical_joint" type="fixed">
-			<origin xyz="0 0 0" rpy="-1.57 0 -1.57" />
-			<parent link="camera_rgb_frame" />
-			<child link="camera_rgb_optical_frame" />
-		</joint>
-		<link name="camera_rgb_optical_frame">
-			<inertial>
-			<mass value="0.001" />
-			<origin xyz="0 0 0" />
-			<inertia ixx="0.0001" ixy="0.0" ixz="0.0"
-				iyy="0.0001" iyz="0.0"
-				izz="0.0001" />
-			</inertial>
-		</link>
+		<link name="camera_optical_frame"/>
 		<gazebo reference="camera_link">
 			<sensor name="kinect" type="depth">
@@ -91,11 +41,11 @@
 					<horizontal_fov>1.047198</horizontal_fov>
 					<image>
-						<width>128</width>
-						<height>128</height>
+						<width>640</width>
+						<height>480</height>
 						<format>R8G8B8</format>
 					</image>
 					<clip>
 						<near>0.05</near>
-						<far>4</far>
+						<far>20</far>
 					</clip>
 				</camera>
@@ -110,5 +60,5 @@
 					<depthImageInfoTopicName>/kinect/depth/camera_info</depthImageInfoTopicName>
 					<pointCloudTopicName>/kinect/depth/points</pointCloudTopicName>
-					<frameName>camera_link</frameName>
+					<frameName>camera_optical_frame</frameName>
 					<pointCloudCutoff>0.05</pointCloudCutoff>
 					<pointCloudCutoffMax>20</pointCloudCutoffMax>

Commit message: update

File: blattoidea/urdf/DiffDrive.xacro (robot description, xacro)
@@ -12,5 +12,5 @@
 				</actuator>
 			</transmission>
-			<transmission name="r_tran">
+		<transmission name="r_tran">
 			<type>transmission_interface/SimpleTransmission</type>
 			<joint name="rw_joint">
@@ -23,5 +23,5 @@
 		</transmission>
 		<gazebo>
-			<plugin ns="DiffDrive" name="differential_drive_controller"
+			<plugin name="differential_drive_controller"
 				filename="libgazebo_ros_diff_drive.so">
 				<alwaysOn>true</alwaysOn>
@@ -31,15 +31,15 @@
 				<wheelSeparation>0.44</wheelSeparation>
 				<wheelDiameter>0.1651</wheelDiameter>
-				<torque>1.41</torque>
 				<commandTopic>cmd_vel</commandTopic>
-				<odometryTopic>odom</odometryTopic>
+				<odometryTopic>/odom</odometryTopic>
 				<odometryFrame>odom</odometryFrame>
 				<robotBaseFrame>base_footprint</robotBaseFrame>
 				<publishWheelJointState>true</publishWheelJointState>
+				<robotNamespace>/</robotNamespace>
 				<rosDebugLevel></rosDebugLevel>
 				<publishWheelTF>false</publishWheelTF>
 				<publishOdomTF>true</publishOdomTF>
 				<wheelAcceleration>0</wheelAcceleration>
-				<wheelTorque>5</wheelTorque>
+				<wheelTorque>1.41</wheelTorque>
 				<odometrySource>world</odometrySource>
 				<publishTf>1</publishTf>

File: blattoidea/urdf/blattoidea.urdf.xacro (robot description, xacro)
@@ -102,5 +102,5 @@
     <axis
       xyz="1 0 0" />
-      <dynamics damping="5.0" friction="10.0"/>
+      <dynamics damping="0.0" friction="0.0"/>
   </joint>
   <link
@@ -156,5 +156,5 @@
     <axis
       xyz="-1 0 0" />
-      <dynamics damping="5.0" friction="10.0"/>
+      <dynamics damping="0.0" friction="0.0"/>
   </joint>
   <link
@@ -200,5 +200,5 @@
   <joint
     name="r_caster_joint"
-    type="continuous">
+    type="fixed">
     <origin
       xyz="-0.15936 -0.14 -0.0051144"
@@ -254,5 +254,5 @@
   <joint
     name="rc_wheel_joint"
-    type="continuous">
+    type="fixed">
     <origin
       xyz="0 -0.049133 0.02245"
@@ -264,5 +264,5 @@
     <axis
       xyz="1 0 0" />
-      <dynamics damping="0.05" friction="0.1"/>
+      <dynamics damping="0.0" friction="0.0"/>
   </joint>
   <link
@@ -308,5 +308,5 @@
   <joint
     name="l_caster_joint"
-    type="continuous">
+    type="fixed">
     <origin
       xyz="-0.15936 0.14 -0.0051144"
@@ -362,5 +362,5 @@
   <joint
     name="lc_wheel_joint"
-    type="continuous">
+    type="fixed">
     <origin
       xyz="0 -0.049133 0.02245"
@@ -372,80 +372,5 @@
     <axis
       xyz="-1 0 0" />
-      <dynamics damping="0.05" friction="0.1"/>
-  </joint>
-<joint name="base_camera_joint" type="fixed">
-				<axis xyz="1 0 0" />
-				<origin xyz="0.17 0.0 0.17" rpy="0 0 0" />
-				<parent link="base_link" />
-				<child link="camera_link" />
-			  </joint>
-		<link name="camera_link">
-			<inertial>
-				<mass value="0.01" />
-				<origin xyz="0 0 0" />
-				<inertia ixx="0.001" ixy="0.0" ixz="0.0"
-					iyy="0.001" iyz="0.0"
-					izz="0.001" />
-			</inertial>
-				<visual>
-				<origin xyz=" 0 0 0 " rpy="0 0 0" />
-				<geometry>
-					<mesh filename="package://blattoidea/meshes/kinect.dae"/>
-				</geometry>
-			</visual>
-			<collision>
-				<origin xyz="0.0 0.0 0.0" rpy="0 0 0" />
-				<geometry>
-					<box size="0.0730 .2760 0.0720"/>
-				</geometry>
-			</collision>
-		</link>
-		<joint name="camera_optical_joint" type="fixed">
-			<origin xyz="0 0 0" rpy="-1.57 0 -1.57" />
-			<parent link="camera_link" />
-			<child link="camera_optical_frame" />
-		</joint>
-		<link name="camera_optical_frame"/>
-		<gazebo reference="camera_optical_frame"/>
-		<gazebo reference="camera_link">
-			<sensor name="kinect" type="depth">
-				<update_rate>30</update_rate>
-				<camera>
-					<horizontal_fov>1.047198</horizontal_fov>
-					<image>
-						<width>640</width>
-						<height>480</height>
-						<format>R8G8B8</format>
-					</image>
-					<clip>
-						<near>0.05</near>
-						<far>20</far>
-					</clip>
-				</camera>
-				<plugin name="depth_controller" filename="libgazebo_ros_openni_kinect.so">
-					<baseline>0.2</baseline>
-					<alwaysOn>true</alwaysOn>
-					<updateRate>30.0</updateRate>
-					<cameraName>kinect_ir</cameraName>
-					<imageTopicName>/kinect/color/image_raw</imageTopicName>
-					<cameraInfoTopicName>/kinect/color/camera_info</cameraInfoTopicName>
-					<depthImageTopicName>/kinect/depth/image_raw</depthImageTopicName>
-					<depthImageInfoTopicName>/kinect/depth/camera_info</depthImageInfoTopicName>
-					<pointCloudTopicName>/kinect/depth/points</pointCloudTopicName>
-					<frameName>camera_optical_frame</frameName>
-					<pointCloudCutoff>0.05</pointCloudCutoff>
-					<pointCloudCutoffMax>20</pointCloudCutoffMax>
-					<distortionK1>0.0</distortionK1>
-					<distortionK2>0.0</distortionK2>
-					<distortionK3>0.0</distortionK3>
-					<distortionT1>0.0</distortionT1>
-					<distortionT2>0.0</distortionT2>
-					<CxPrime>0</CxPrime>
-					<Cx>0</Cx>
-					<Cy>0</Cy>
-					<focalLength>0</focalLength>
-					<hackBaseline>0</hackBaseline>
-				</plugin>
-			</sensor>
-		</gazebo>
+      <dynamics damping="0.0" friction="0.0"/>
+  </joint>
 </robot>

File: blattoidea/urdf/blattoidea_gazebo.urdf.xacro (robot description, xacro)
@@ -10,8 +10,8 @@
 	<xacro:include filename="$(find blattoidea)/urdf/DiffDrive.xacro"/>
 	<xacro:DiffDrive/>
-	<!--<xacro:include filename="$(find blattoidea)/urdf/kinect.xacro"/>
-	<xacro:kinect/>-->
-	<!--<xacro:include filename="$(find blattoidea)/urdf/camera.xacro"/>
-	<xacro:rgb_camera/>-->
+	<xacro:include filename="$(find blattoidea)/urdf/kinect.xacro"/>
+	<xacro:kinect/>
+	<xacro:include filename="$(find blattoidea)/urdf/camera.xacro"/>
+	<xacro:rgb_camera/>
 	<xacro:include filename="$(find blattoidea)/urdf/hokuyo.xacro"/>
 	<xacro:laser name="base_laser" parent="base_link" xyz="0.17 0.0 0.085" rpy="3.14 0 0" meshes="package://gazebo_plugins/test/multi_robot_scenario/meshes/laser"/>

File: blattoidea/urdf/camera.xacro (robot description, xacro)
@@ -94,4 +94,5 @@
 			<distortionT1>0.0</distortionT1>
 			<distortionT2>0.0</distortionT2>
+			<robotNamespace>/</robotNamespace>
 		      </plugin>
 		    </sensor>

File: blattoidea/urdf/hokuyo.xacro (robot description, xacro)
@@ -48,5 +48,5 @@
           </ray>
           <plugin name="laser" filename="libgazebo_ros_laser.so" >
-              <!--<robotNamespace></robotNamespace>-->
+              <robotNamespace>/</robotNamespace>
             <topicName>scan</topicName>
             <frameName>base_laser</frameName>

Commit message: update

File: blattoidea/urdf/DiffDrive.xacro (robot description, xacro)
@@ -32,5 +32,5 @@
 				<wheelDiameter>0.1651</wheelDiameter>
 				<commandTopic>cmd_vel</commandTopic>
-				<odometryTopic>/odom</odometryTopic>
+				<odometryTopic>odom</odometryTopic>
 				<odometryFrame>odom</odometryFrame>
 				<robotBaseFrame>base_footprint</robotBaseFrame>

File: blattoidea/urdf/blattoidea_gazebo.urdf.xacro (robot description, xacro)
@@ -17,4 +17,4 @@
 	<xacro:rgb_camera/> -->
 	<xacro:include filename="$(find blattoidea)/urdf/hokuyo.xacro"/>
-	<xacro:laser name="base_laser" parent="base_link" xyz="0.17 0.0 0.085" rpy="3.14 0 0" meshes="package://gazebo_plugins/test/multi_robot_scenario/meshes/laser"/>
+	<xacro:laser name="base_laser" parent="base_link" xyz="0.17 0.0 0.085" rpy="3.14 0 0" meshes="package://gazebo_plugins/test/multi_robot_scenario/meshes/laser" gpu="false"/>
 </robot>

File: blattoidea/urdf/hokuyo.xacro (robot description, xacro)
@@ -2,5 +2,5 @@
 <robot xmlns:xacro="http://www.ros.org/wiki/xacro">
 <!-- Front Laser -->
-<xacro:macro name="laser" params="name parent xyz rpy meshes" >
+<xacro:macro name="laser" params="name parent xyz rpy meshes gpu" >
   <joint name="${parent}_${name}_joint" type="fixed">
       <axis xyz="0 0 1" />
@@ -47,9 +47,16 @@
             </range>
           </ray>
+					<xacro:unless value="${gpu}">
           <plugin name="laser" filename="libgazebo_ros_laser.so" >
-              <robotNamespace>/</robotNamespace>
-            <topicName>scan</topicName>
-            <frameName>base_laser</frameName>
+            <topicName>/scan</topicName>
+            <frameName>${name}</frameName>
           </plugin>
+          </xacro:unless>
+          <xacro:if value="${gpu}">
+          <plugin name="laser" filename="libgazebo_ros_gpu_laser.so" >
+            <topicName>/scan</topicName>
+            <frameName>${name}</frameName>
+          </plugin>
+          </xacro:if>
           <!--
           <plugin name="laser" filename="libRayPlugin.so" />
